Commit message: Changed the whole structure of the docking algorithm. Steps to docking are: 1. Travel to far detection zone 2. Spin until AprilTag is found 3. Travel to near detection zone 4. Spin until Apriltag is found 5. Dock

File: simulation_launch/urdf/mobile_bot.urdf (robot description, URDF)
Before this commit: robot mobile_bot, 9 links, 8 joints
Links:
- added link lidar_link, mass 0.1; collision cylinder length=0.07 radius=0.1; visual cylinder length=0.07 radius=0.1
Joints:
- added joint lidar_joint: type fixed, parent base_link, child lidar_link, origin xyz=0 0 0.185 rpy=0 0 0

File: simulation_launch/urdf/mobile_bot.xacro (robot description, xacro)
@@ -218,9 +218,9 @@
             <right_joint>drive_wheel_r_joint</right_joint>
             <!-- kinematics -->
-            <wheel_separation>0.44</wheel_separation>
-            <wheel_diameter>0.14</wheel_diameter>
+            <wheel_separation>0.35</wheel_separation>
+            <wheel_diameter>0.2</wheel_diameter>
             <!-- limits -->
-            <max_wheel_torque>100</max_wheel_torque>
-            <max_wheel_acceleration>10.0</max_wheel_acceleration>
+            <max_wheel_torque>20</max_wheel_torque>
+            <max_wheel_acceleration>1.0</max_wheel_acceleration>
             <!-- input -->
             <!-- subscribe to the /cmd_vel topic-->
@@ -239,4 +239,58 @@
             <robot_base_frame>base_footprint</robot_base_frame>
         </plugin>
+    </gazebo>
+    <link name="lidar_link">
+        <visual>
+            <origin xyz="0 0 0" rpy="0 0 0"/>
+            <geometry>
+                <cylinder radius="${lidar_radius}" length="${lidar_height}"/>
+            </geometry>
+        </visual>
+        <collision>
+            <origin xyz="0 0 0" rpy="0 0 0"/>
+            <geometry>
+                <cylinder radius="${lidar_radius}" length="${lidar_height}"/>
+            </geometry>
+        </collision>
+        <xacro:cylinder_inertia m="0.1" r="${lidar_radius}" h="${lidar_height}"/>
+    </link>
+    <joint name="lidar_joint" type="fixed">
+        <parent link="base_link"/>
+        <child link="lidar_link"/>
+        <origin xyz="0 0 ${(base_height/2)+(lidar_height/2)}" rpy="0 0 0"/>
+    </joint>
+    <gazebo reference="lidar_link">
+        <sensor name="lidar" type="ray">
+        <always_on>true</always_on>
+        <visualize>true</visualize>
+        <update_rate>5</update_rate>
+        <ray>
+            <scan>
+            <horizontal>
+                <samples>360</samples>
+                <resolution>1.000000</resolution>
+                <min_angle>0.000000</min_angle>
+                <max_angle>6.280000</max_angle>
+            </horizontal>
+            </scan>
+            <range>
+            <min>0.120000</min>
+            <max>6.0</max>
+            <resolution>0.015000</resolution>
+            </range>
+            <noise>
+            <type>gaussian</type>
+            <mean>0.0</mean>
+            <stddev>0.01</stddev>
+            </noise>
+        </ray>
+        <plugin name="scan" filename="libgazebo_ros_ray_sensor.so">
+            <ros>
+            <remapping>~/out:=scan</remapping>
+            </ros>
+            <output_type>sensor_msgs/LaserScan</output_type>
+            <frame_name>lidar_link</frame_name>
+        </plugin>
+        </sensor>
     </gazebo>
     <link name="camera_link">
